File: Lab 6/Lab 4 555 timer/Lab 4 555 timer.kicad_pcb (KiCad board)
At the start: 2 copper layers, 45.7 x 50.8 mm, 10 parts, among them J1 Conn_01x02_Male, U1 NE555D

Commit message: Lab 7 push
Routing:
- net +9V: track 58.6 -> 54.3 mm
Changed lines of the file:
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@@
   )
   (setup
+    (stackup
+      (layer "F.SilkS" (type "Top Silk Screen"))
+      (layer "F.Paste" (type "Top Solder Paste"))
+      (layer "F.Mask" (type "Top Solder Mask") (thickness 0.01))
+      (layer "F.Cu" (type "copper") (thickness 0.035))
+      (layer "dielectric 1" (type "core") (thickness 1.51) (material "FR4") (epsilon_r 4.5) (loss_tangent 0.02))
+      (layer "B.Cu" (type "copper") (thickness 0.035))
+      (layer "B.Mask" (type "Bottom Solder Mask") (thickness 0.01))
+      (layer "B.Paste" (type "Bottom Solder Paste"))
+      (layer "B.SilkS" (type "Bottom Silk Screen"))
+      (copper_finish "None")
+      (dielectric_constraints no)
+    )
     (pad_to_mask_clearance 0)
     (pcbplotparams
@@
   (segment (start 134.392936 88.672936) (end 131.35 88.672936) (width 0.25) (layer "F.Cu") (net 4))
   (segment (start 151.545 79.595) (end 152.4 78.74) (width 0.25) (layer "F.Cu") (net 5))
-  (segment (start 154.94 71.12) (end 160.02 76.2) (width 0.25) (layer "F.Cu") (net 5))
   (segment (start 156.65 78.74) (end 154.94 78.74) (width 0.25) (layer "F.Cu") (net 5))
-  (segment (start 160.02 78.15) (end 158.04 80.13) (width 0.25) (layer "F.Cu") (net 5))
+  (segment (start 154.94 78.74) (end 154.94 66.04) (width 0.25) (layer "F.Cu") (net 5))
   (segment (start 152.4 78.74) (end 154.94 78.74) (width 0.25) (layer "F.Cu") (net 5))
   (segment (start 142.24 92.8775) (end 142.24 83.5) (width 0.25) (layer "F.Cu") (net 5))
   (segment (start 151.545 79.595) (end 147.285 79.595) (width 0.25) (layer "F.Cu") (net 5))
-  (segment (start 160.02 76.2) (end 160.02 78.15) (width 0.25) (layer "F.Cu") (net 5))
   (segment (start 142.24 83.5) (end 142.335 83.405) (width 0.25) (layer "F.Cu") (net 5))
   (segment (start 140.2 94.9175) (end 142.24 92.8775) (width 0.25) (layer "F.Cu") (net 5))
-  (segment (start 154.94 66.04) (end 154.94 71.12) (width 0.25) (layer "F.Cu") (net 5))
   (segment (start 156.65 78.74) (end 158.04 80.13) (width 0.25) (layer "F.Cu") (net 5))
   (via (at 142.24 86.36) (size 0.8) (drill 0.4) (layers "F.Cu" "B.Cu") (net 5))
